File: kicad/obs-studio-controller/obs-studio-controller.kicad_sch (KiCad schematic)
At the start: 17 parts

Commit message: Placed parts in pcb layout, nothing moved yet
Parts:
- gave numbers to parts that had none: 17

Commit message: Routing complete
Parts:
- removed D1: LED5V, LED_SMD:LED_0603_1608Metric, symbol Device:LED
- removed R3: 1k, Resistor_SMD:R_0402_1005Metric, symbol Device:R
- added J6: GPIO, Connector_PinSocket_2.54mm:PinSocket_1x06_P2.54mm_Vertical, symbol Connector_Generic:Conn_01x06
- added J7: WS2812, Connector_PinSocket_2.54mm:PinSocket_1x03_P2.54mm_Vertical, symbol Connector_Generic:Conn_01x03
Connections:
- net +5V: now also J7.3 (Pin_3)
- net EXT_SENSE: now also U1.7 (IO35)
- net GND: now also J7.1 (Pin_1)
- net IO26: now reaches U1.11 (IO26)
- net IO26: now also J6.5 (Pin_5)
- net IO27: now reaches U1.12 (IO27)
- net IO27: now also J6.4 (Pin_4)
- net BTN_IN3: now reaches U1.27 (IO16)
- net BTN_IN4: now reaches U1.28 (IO17)
- net IO5: now reaches U1.29 (IO5)
- net IO5: now also J6.6 (Pin_6), J7.2 (Pin_2)
- net IO34: now reaches U1.6 (IO34)
- net IO34: now also J6.1 (Pin_1)
- net IO32: now reaches U1.8 (IO32)
- net IO32: now also J6.3 (Pin_3)
- net IO33: now reaches U1.9 (IO33)
- net IO33: now also J6.2 (Pin_2)
- net +5VUSB renamed VEXT
Other:
- added sheet AMS1117-5V-3v3 (voltage_regulator.kicad_sch)
- sheet Buttons ports: added IN_3, IN_4; removed none
- moved on the sheet: J1, JP1

Commit message: Updated production files
Parts:
- C1: LCSC (none) -> C19702
- C2: footprint Capacitor_SMD:C_0603_1608Metric -> Capacitor_SMD:C_0402_1005Metric; LCSC (none) -> C1525
- J1, J2, J3, J6, J7: LCSC (none) -> DNP
- R2: LCSC C25086 -> C25741
- R6, R7, R8, R9: LCSC (none) -> C22775
- U1: LCSC (none) -> C701342
Changed lines of the file:
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@@
+      (effects (font (size 1.27 1.27)) hide)
+    )
+    (property "LCSC" "C19702" (id 5) (at 140.335 39.37 0)
       (effects (font (size 1.27 1.27)) hide)
     )
@@
     )
     (property "LCSC Part #" "DNP" (id 4) (at 212.725 102.87 90)
+      (effects (font (size 1.27 1.27)) hide)
+    )
+    (property "LCSC" "DNP" (id 5) (at 215.265 112.395 0)
       (effects (font (size 1.27 1.27)) hide)
     )
@@
     )
     (property "LCSC Part #" "C701343" (id 4) (at 144.145 92.075 0)
+      (effects (font (size 1.27 1.27)) hide)
+    )
+    (property "LCSC" "C701342" (id 5) (at 132.715 57.785 0)
       (effects (font (size 1.27 1.27)) hide)
     )
@@
       (effects (font (size 1.27 1.27)) hide)
     )
+    (property "LCSC" "C22775" (id 5) (at 182.88 102.235 0)
+      (effects (font (size 1.27 1.27)) hide)
+    )
     (pin "1")
     (pin "2")
@@
       (effects (font (size 1.27 1.27)) hide)
     )
-    (property "LCSC" "C25086" (id 4) (at 36.83 153.67 0)
+    (property "LCSC" "C25741" (id 4) (at 36.83 153.67 0)
       (effects (font (size 1.27 1.27)) hide)
     )
@@
       (effects (font (size 1.27 1.27)) hide)
     )
+    (property "LCSC" "DNP" (id 5) (at 163.195 21.59 0)
+      (effects (font (size 1.27 1.27)) hide)
+    )
     (pin "1")
     (pin "2")
@@
       (effects (font (size 1.27 1.27)) hide)
     )
+    (property "LCSC" "DNP" (id 5) (at 92.71 170.18 0)
+      (effects (font (size 1.27 1.27)) hide)
+    )
     (pin "1")
     (pin "2")
@@
       (effects (font (size 1.27 1.27)) hide)
     )
+    (property "LCSC" "DNP" (id 5) (at 199.39 75.565 0)
+      (effects (font (size 1.27 1.27)) hide)
+    )
     (pin "1")
     (pin "2")
@@
     )
     (property "LCSC Part #" "DNP" (id 4) (at 167.64 99.695 90)
+      (effects (font (size 1.27 1.27)) hide)
+    )
+    (property "LCSC" "DNP" (id 5) (at 170.18 109.22 0)
       (effects (font (size 1.27 1.27)) hide)
     )
@@
       (effects (font (size 1.27 1.27)) hide)
     )
+    (property "LCSC" "C22775" (id 5) (at 182.88 94.615 0)
+      (effects (font (size 1.27 1.27)) hide)
+    )
     (pin "1")
     (pin "2")
@@
     (property "Reference" "C2" (id 0) (at 137.795 54.61 90))
     (property "Value" "100n" (id 1) (at 141.605 54.61 90))
-    (property "Footprint" "Capacitor_SMD:C_0603_1608Metric" (id 2) (at 144.145 49.8348 0)
+    (property "Footprint" "Capacitor_SMD:C_0402_1005Metric" (id 2) (at 144.145 49.8348 0)
       (effects (font (size 1.27 1.27)) hide)
     )
@@
       (effects (font (size 1.27 1.27)) hide)
     )
+    (property "LCSC" "C1525" (id 5) (at 137.795 54.61 0)
+      (effects (font (size 1.27 1.27)) hide)
+    )
     (pin "1")
     (pin "2")
@@
       (effects (font (size 1.27 1.27)) hide)
     )
+    (property "LCSC" "C22775" (id 5) (at 182.88 99.695 0)
+      (effects (font (size 1.27 1.27)) hide)
+    )
     (pin "1")
     (pin "2")
@@
     )
     (property "LCSC Part #" "C22775" (id 4) (at 179.07 99.695 0)
+      (effects (font (size 1.27 1.27)) hide)
+    )
+    (property "LCSC" "C22775" (id 5) (at 182.88 97.155 0)
       (effects (font (size 1.27 1.27)) hide)
     )
@@
     )
     (path "/e85a09df-376b-48e1-b2a9-fe146fc16152"
-      (reference "C2") (unit 1) (value "100n") (footprint "Capacitor_SMD:C_0603_1608Metric")
+      (reference "C2") (unit 1) (value "100n") (footprint "Capacitor_SMD:C_0402_1005Metric")
     )
     (path "/14aa7fc0-62ed-4ece-b8c9-769201a8d33d/f6b3ba70-2bc2-444d-be91-c029c0109157"
