File: kicad/obs-studio-controller/obs-studio-controller.kicad_sch (KiCad schematic)
At the start: 17 parts, among them J1 PWR_SWITCH, J2 EXT_PWR, J3 LEDS, J6 GPIO, J7 WS2812, U1 ESP32-WROOM-32

Commit message: Actually connect rotary encoder
Parts:
- removed J1: PWR_SWITCH, Connector_PinSocket_2.54mm:PinSocket_1x02_P2.54mm_Vertical, symbol Connector_Generic:Conn_01x02
- removed J2: EXT_PWR, Connector_PinSocket_2.54mm:PinSocket_1x03_P2.54mm_Vertical, symbol Connector_Generic:Conn_01x03
- removed J6: GPIO, Connector_PinSocket_2.54mm:PinSocket_1x06_P2.54mm_Vertical, symbol Connector_Generic:Conn_01x06
- removed JP1: SolderJumper_2_Open, Jumper:SolderJumper-2_P1.3mm_Open_RoundedPad1.0x1.5mm, symbol Jumper:SolderJumper_2_Open
- removed R1: 30k, Resistor_SMD:R_0603_1608Metric, symbol Device:R
- removed R2: 100k, Resistor_SMD:R_0402_1005Metric, symbol Device:R
Connections:
- net EXT_SENSE is gone; now on net ROT3_DT: U1.7 (IO35)
- net IO26 is gone; now on net ROT1_CLK: U1.11 (IO26)
- net IO27 is gone; now on net ROT1_DT: U1.12 (IO27)
- net IO32 is gone; now on net ROT2_CLK: U1.8 (IO32)
- net IO33 is gone; now on net ROT2_DT: U1.9 (IO33)
- net IO34 is gone; now on net ROT3_CLK: U1.6 (IO34)
- net ROT4_CLK: now also U1.4 (SENSOR_VP)
- net ROT4_DT: now also U1.5 (SENSOR_VN)
