File: kicad/obs-studio-controller/rotary.kicad_sch (KiCad schematic)
At the start: 4 parts

Commit message: Placed parts in pcb layout, nothing moved yet
Parts:
- SW1: renamed from SW?; footprint (none) -> Rotary_Encoder:RotaryEncoder_Alps_EC12E-Switch_Vertical_H20mm_CircularMountingHoles; LCSC (none) -> C129727
- gave numbers to parts that had none: 3
Changed lines of the file:
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@@
   (symbol (lib_id "Device:R") (at 34.925 45.085 0) (unit 1)
     (in_bom yes) (on_board yes)
-    (property "Reference" "R?" (id 0) (at 36.703 43.9166 0)
+    (property "Reference" "R11" (id 0) (at 36.703 43.9166 0)
       (effects (font (size 1.27 1.27)) (justify left))
     )
@@
   (symbol (lib_id "Device:R") (at 34.925 32.385 0) (unit 1)
     (in_bom yes) (on_board yes)
-    (property "Reference" "R?" (id 0) (at 36.703 31.2166 0)
+    (property "Reference" "R10" (id 0) (at 36.703 31.2166 0)
       (effects (font (size 1.27 1.27)) (justify left))
     )
@@
   (symbol (lib_id "Device:RotaryEncoder_Switch") (at 45.72 38.735 0) (unit 1)
     (in_bom yes) (on_board yes)
-    (property "Reference" "SW?" (id 0) (at 55.88 48.26 0))
+    (property "Reference" "SW1" (id 0) (at 55.88 48.26 0))
     (property "Value" "RotaryEncoder_Switch" (id 1) (at 52.705 45.72 0))
-    (property "Footprint" "" (id 2) (at 41.91 34.671 0)
+    (property "Footprint" "Rotary_Encoder:RotaryEncoder_Alps_EC12E-Switch_Vertical_H20mm_CircularMountingHoles" (id 2) (at 41.91 34.671 0)
       (effects (font (size 1.27 1.27)) hide)
     )
     (property "Datasheet" "~" (id 3) (at 45.72 32.131 0)
+      (effects (font (size 1.27 1.27)) hide)
+    )
+    (property "LCSC" "C129727" (id 4) (at 45.72 38.735 0)
       (effects (font (size 1.27 1.27)) hide)
     )
@@
   (symbol (lib_id "Device:R") (at 55.245 32.385 0) (unit 1)
     (in_bom yes) (on_board yes)
-    (property "Reference" "R?" (id 0) (at 57.023 31.2166 0)
+    (property "Reference" "R12" (id 0) (at 57.023 31.2166 0)
       (effects (font (size 1.27 1.27)) (justify left))
     )

Commit message: Added rotary 3d model, discovered that the lcsc part number is wrong
Parts:
- SW1: footprint Rotary_Encoder:RotaryEncoder_Alps_EC12E-Switch_Vertical_H20mm_CircularMountingHoles -> custom:RotaryEncoder_Alps_EC12E-Switch_Vertical_H20mm_CircularMountingHoles
Changed lines of the file:
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@@
     (property "Reference" "SW1" (id 0) (at 55.88 48.26 0))
     (property "Value" "RotaryEncoder_Switch" (id 1) (at 52.705 45.72 0))
-    (property "Footprint" "Rotary_Encoder:RotaryEncoder_Alps_EC12E-Switch_Vertical_H20mm_CircularMountingHoles" (id 2) (at 41.91 34.671 0)
+    (property "Footprint" "custom:RotaryEncoder_Alps_EC12E-Switch_Vertical_H20mm_CircularMountingHoles" (id 2) (at 41.91 34.671 0)
       (effects (font (size 1.27 1.27)) hide)
     )
