File: kicad/obs-studio-controller/buttons.kicad_sch (KiCad schematic)
At the start: 7 parts

Commit message: Placed parts in pcb layout, nothing moved yet
Parts:
- gave numbers to parts that had none: 7
Changed lines of the file:
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@@
   (symbol (lib_id "Power_Protection:USBLC6-4SC6") (at 135.255 41.91 0) (unit 1)
     (in_bom yes) (on_board yes) (fields_autoplaced)
-    (property "Reference" "U?" (id 0) (at 138.0237 30.3235 0)
+    (property "Reference" "U2" (id 0) (at 138.0237 30.3235 0)
       (effects (font (size 1.27 1.27)) (justify left))
     )
@@
   (symbol (lib_id "power:+3V3") (at 135.255 31.75 0) (unit 1)
     (in_bom yes) (on_board yes)
-    (property "Reference" "#PWR?" (id 0) (at 135.255 35.56 0)
+    (property "Reference" "#PWR0120" (id 0) (at 135.255 35.56 0)
       (effects (font (size 1.27 1.27)) hide)
     )
@@
   (symbol (lib_id "Diode:BAV99") (at 62.23 78.74 0) (unit 1)
     (in_bom yes) (on_board yes) (fields_autoplaced)
-    (property "Reference" "D?" (id 0) (at 62.23 72.39 0))
+    (property "Reference" "D3" (id 0) (at 62.23 72.39 0))
     (property "Value" "BAV99" (id 1) (at 62.23 74.93 0))
     (property "Footprint" "Package_TO_SOT_SMD:SOT-23" (id 2) (at 62.23 91.44 0)
@@
   (symbol (lib_id "Diode:BAV99") (at 100.33 78.74 0) (unit 1)
     (in_bom yes) (on_board yes) (fields_autoplaced)
-    (property "Reference" "D?" (id 0) (at 100.33 72.39 0))
+    (property "Reference" "D5" (id 0) (at 100.33 72.39 0))
     (property "Value" "BAV99" (id 1) (at 100.33 74.93 0))
     (property "Footprint" "Package_TO_SOT_SMD:SOT-23" (id 2) (at 100.33 91.44 0)
@@
   (symbol (lib_id "Connector_Generic:Conn_02x08_Odd_Even") (at 76.835 46.355 0) (unit 1)
     (in_bom yes) (on_board yes) (fields_autoplaced)
-    (property "Reference" "J?" (id 0) (at 78.105 33.4985 0))
+    (property "Reference" "J5" (id 0) (at 78.105 33.4985 0))
     (property "Value" "Conn_02x08_Odd_Even" (id 1) (at 78.105 36.2736 0))
     (property "Footprint" "Connector_PinHeader_2.54mm:PinHeader_2x08_P2.54mm_Vertical" (id 2) (at 76.835 46.355 0)
@@
   (symbol (lib_id "Diode:BAV99") (at 41.91 78.74 0) (unit 1)
     (in_bom yes) (on_board yes) (fields_autoplaced)
-    (property "Reference" "D?" (id 0) (at 41.91 72.39 0))
+    (property "Reference" "D2" (id 0) (at 41.91 72.39 0))
     (property "Value" "BAV99" (id 1) (at 41.91 74.93 0))
     (property "Footprint" "Package_TO_SOT_SMD:SOT-23" (id 2) (at 41.91 91.44 0)
@@
   (symbol (lib_id "power:+3V3") (at 135.89 69.85 0) (unit 1)
     (in_bom yes) (on_board yes)
-    (property "Reference" "#PWR?" (id 0) (at 135.89 73.66 0)
+    (property "Reference" "#PWR0119" (id 0) (at 135.89 73.66 0)
       (effects (font (size 1.27 1.27)) hide)
     )
@@
   (symbol (lib_id "Power_Protection:USBLC6-4SC6") (at 135.89 80.01 0) (unit 1)
     (in_bom yes) (on_board yes) (fields_autoplaced)
-    (property "Reference" "U?" (id 0) (at 138.6587 68.4235 0)
+    (property "Reference" "U3" (id 0) (at 138.6587 68.4235 0)
       (effects (font (size 1.27 1.27)) (justify left))
     )
@@
   (symbol (lib_id "Diode:BAV99") (at 81.28 78.74 0) (unit 1)
     (in_bom yes) (on_board yes) (fields_autoplaced)
-    (property "Reference" "D?" (id 0) (at 81.28 72.39 0))
+    (property "Reference" "D4" (id 0) (at 81.28 72.39 0))
     (property "Value" "BAV99" (id 1) (at 81.28 74.93 0))
     (property "Footprint" "Package_TO_SOT_SMD:SOT-23" (id 2) (at 81.28 91.44 0)
@@
   (symbol (lib_id "power:GND") (at 135.255 52.07 0) (unit 1)
     (in_bom yes) (on_board yes)
-    (property "Reference" "#PWR?" (id 0) (at 135.255 58.42 0)
+    (property "Reference" "#PWR0121" (id 0) (at 135.255 58.42 0)
       (effects (font (size 1.27 1.27)) hide)
     )
@@
   (symbol (lib_id "power:GND") (at 135.89 90.17 0) (unit 1)
     (in_bom yes) (on_board yes)
-    (property "Reference" "#PWR?" (id 0) (at 135.89 96.52 0)
+    (property "Reference" "#PWR0118" (id 0) (at 135.89 96.52 0)
       (effects (font (size 1.27 1.27)) hide)
     )

Commit message: Routing complete
Parts:
- J5: value Conn_02x08_Odd_Even -> BUTTONS
Connections:
- net IN_1: no longer J5.6 (Pin_6), J5.8 (Pin_8)
- net IN_2: now also J5.6 (Pin_6), J5.8 (Pin_8); no longer J5.10 (Pin_10), J5.12 (Pin_12), J5.14 (Pin_14), J5.16 (Pin_16)
- new net IN_3: J5.10 (Pin_10), J5.12 (Pin_12)
- new net IN_4: J5.14 (Pin_14), J5.16 (Pin_16)
Changed lines of the file:
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@@
     (effects (font (size 1.27 1.27)) (justify left))
   )
-  (hierarchical_label "IN_1" (shape input) (at 84.455 46.355 0)
+  (hierarchical_label "IN_2" (shape input) (at 84.455 46.355 0)
     (effects (font (size 1.27 1.27)) (justify left))
   )
@@
     (effects (font (size 1.27 1.27)) (justify right))
   )
-  (hierarchical_label "IN_2" (shape input) (at 84.455 51.435 0)
+  (hierarchical_label "IN_3" (shape input) (at 84.455 51.435 0)
     (effects (font (size 1.27 1.27)) (justify left))
   )
@@
     (effects (font (size 1.27 1.27)) (justify left))
   )
-  (hierarchical_label "IN_1" (shape input) (at 84.455 43.815 0)
-    (effects (font (size 1.27 1.27)) (justify left))
-  )
-  (hierarchical_label "IN_2" (shape input) (at 84.455 53.975 0)
+  (hierarchical_label "IN_2" (shape input) (at 84.455 43.815 0)
+    (effects (font (size 1.27 1.27)) (justify left))
+  )
+  (hierarchical_label "IN_4" (shape input) (at 84.455 53.975 0)
     (effects (font (size 1.27 1.27)) (justify left))
   )
@@
     (effects (font (size 1.27 1.27)) (justify left))
   )
-  (hierarchical_label "IN_2" (shape input) (at 84.455 48.895 0)
+  (hierarchical_label "IN_3" (shape input) (at 84.455 48.895 0)
     (effects (font (size 1.27 1.27)) (justify left))
   )
@@
     (effects (font (size 1.27 1.27)) (justify right))
   )
-  (hierarchical_label "IN_2" (shape input) (at 84.455 56.515 0)
+  (hierarchical_label "IN_4" (shape input) (at 84.455 56.515 0)
     (effects (font (size 1.27 1.27)) (justify left))
   )
@@
     (pin "6")
   )
-  (symbol (lib_id "power:+3V3") (at 135.255 31.75 0) (unit 1)
-    (in_bom yes) (on_board yes)
-    (property "Reference" "#PWR0120" (id 0) (at 135.255 35.56 0)
-      (effects (font (size 1.27 1.27)) hide)
-    )
-    (property "Value" "+3V3" (id 1) (at 135.636 27.3558 0))
-    (property "Footprint" "" (id 2) (at 135.255 31.75 0)
-      (effects (font (size 1.27 1.27)) hide)
-    )
-    (property "Datasheet" "" (id 3) (at 135.255 31.75 0)
-      (effects (font (size 1.27 1.27)) hide)
-    )
-    (pin "1")
-  )
   (symbol (lib_id "Diode:BAV99") (at 62.23 78.74 0) (unit 1)
     (in_bom yes) (on_board yes) (fields_autoplaced)
@@
   (symbol (lib_id "Connector_Generic:Conn_02x08_Odd_Even") (at 76.835 46.355 0) (unit 1)
     (in_bom yes) (on_board yes) (fields_autoplaced)
-    (property "Reference" "J5" (id 0) (at 78.105 33.4985 0))
-    (property "Value" "Conn_02x08_Odd_Even" (id 1) (at 78.105 36.2736 0))
+    (property "Reference" "J5" (id 0) (at 78.105 31.75 0))
+    (property "Value" "BUTTONS" (id 1) (at 78.105 34.29 0))
     (property "Footprint" "Connector_PinHeader_2.54mm:PinHeader_2x08_P2.54mm_Vertical" (id 2) (at 76.835 46.355 0)
       (effects (font (size 1.27 1.27)) hide)
@@
     (pin "9")
   )
+  (symbol (lib_id "power:+3.3V") (at 135.89 69.85 0) (unit 1)
+    (in_bom yes) (on_board yes)
+    (property "Reference" "#PWR0120" (id 0) (at 135.89 73.66 0)
+      (effects (font (size 1.27 1.27)) hide)
+    )
+    (property "Value" "+3.3V" (id 1) (at 137.16 67.31 0)
+      (effects (font (size 1.27 1.27)) (justify left))
+    )
+    (property "Footprint" "" (id 2) (at 135.89 69.85 0)
+      (effects (font (size 1.27 1.27)) hide)
+    )
+    (property "Datasheet" "" (id 3) (at 135.89 69.85 0)
+      (effects (font (size 1.27 1.27)) hide)
+    )
+    (pin "1")
+  )
   (symbol (lib_id "Diode:BAV99") (at 41.91 78.74 0) (unit 1)
     (in_bom yes) (on_board yes) (fields_autoplaced)
@@
     (pin "3")
   )
-  (symbol (lib_id "power:+3V3") (at 135.89 69.85 0) (unit 1)
-    (in_bom yes) (on_board yes)
-    (property "Reference" "#PWR0119" (id 0) (at 135.89 73.66 0)
-      (effects (font (size 1.27 1.27)) hide)
-    )
-    (property "Value" "+3V3" (id 1) (at 136.271 65.4558 0))
-    (property "Footprint" "" (id 2) (at 135.89 69.85 0)
-      (effects (font (size 1.27 1.27)) hide)
-    )
-    (property "Datasheet" "" (id 3) (at 135.89 69.85 0)
-      (effects (font (size 1.27 1.27)) hide)
-    )
-    (pin "1")
-  )
   (symbol (lib_id "Power_Protection:USBLC6-4SC6") (at 135.89 80.01 0) (unit 1)
     (in_bom yes) (on_board yes) (fields_autoplaced)
@@
       (effects (font (size 1.27 1.27)) hide)
     )
+    (pin "1")
+  )
+  (symbol (lib_id "power:+3.3V") (at 135.255 31.75 0) (unit 1)
+    (in_bom yes) (on_board yes)
+    (property "Reference" "#PWR0119" (id 0) (at 135.255 35.56 0)
+      (effects (font (size 1.27 1.27)) hide)
+    )
+    (property "Value" "+3.3V" (id 1) (at 136.525 29.21 0)
+      (effects (font (size 1.27 1.27)) (justify left))
+    )
+    (property "Footprint" "" (id 2) (at 135.255 31.75 0)
+      (effects (font (size 1.27 1.27)) hide)
+    )
+    (property "Datasheet" "" (id 3) (at 135.255 31.75 0)
+      (effects (font (size 1.27 1.27)) hide)
+    )

Commit message: Updated production files
Parts:
- D2, D3, D4, D5: LCSC (none) -> C2500
- J5: LCSC (none) -> DNP
- U2, U3: LCSC (none) -> C558419
Changed lines of the file:
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@@
+      (effects (font (size 1.27 1.27)) hide)
+    )
+    (property "LCSC" "C558419" (id 5) (at 138.0237 30.3235 0)
       (effects (font (size 1.27 1.27)) hide)
     )
@@
       (effects (font (size 1.27 1.27)) hide)
     )
+    (property "LCSC" "C2500" (id 4) (at 62.23 72.39 0)
+      (effects (font (size 1.27 1.27)) hide)
+    )
     (pin "1")
     (pin "2")
@@
     )
     (property "Datasheet" "https://assets.nexperia.com/documents/data-sheet/BAV99_SER.pdf" (id 3) (at 100.33 78.74 0)
+      (effects (font (size 1.27 1.27)) hide)
+    )
+    (property "LCSC" "C2500" (id 4) (at 100.33 72.39 0)
       (effects (font (size 1.27 1.27)) hide)
     )
@@
     )
     (property "LCSC Part #" "DNP" (id 4) (at 76.835 46.355 0)
+      (effects (font (size 1.27 1.27)) hide)
+    )
+    (property "LCSC" "DNP" (id 5) (at 78.105 31.75 0)
       (effects (font (size 1.27 1.27)) hide)
     )
@@
       (effects (font (size 1.27 1.27)) hide)
     )
+    (property "LCSC" "C2500" (id 5) (at 41.91 72.39 0)
+      (effects (font (size 1.27 1.27)) hide)
+    )
     (pin "1")
     (pin "2")
@@
       (effects (font (size 1.27 1.27)) hide)
     )
+    (property "LCSC" "C558419" (id 5) (at 138.6587 68.4235 0)
+      (effects (font (size 1.27 1.27)) hide)
+    )
     (pin "1")
     (pin "2")
@@
       (effects (font (size 1.27 1.27)) hide)
     )
+    (property "LCSC" "C2500" (id 4) (at 81.28 72.39 0)
+      (effects (font (size 1.27 1.27)) hide)
+    )
