File: kicad/obs-studio-controller/usb_c.kicad_sch (KiCad schematic)
At the start: 22 parts

Commit message: Placed parts in pcb layout, nothing moved yet
Parts:
- gave numbers to parts that had none: 22

Commit message: Routing complete
Other:
- removed sheet AMS1117-5V-3v3
Changed lines of the file:
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@@
-    (stroke (width 0) (type default) (color 0 0 0 0))
-  )
-  (wire (pts (xy 50.8 129.54) (xy 53.975 129.54))
     (stroke (width 0) (type default) (color 0 0 0 0))
   )
@@
     (stroke (width 0) (type default) (color 0 0 0 0))
   )
-  (wire (pts (xy 50.8 132.08) (xy 53.975 132.08))
-    (stroke (width 0) (type default) (color 0 0 0 0))
-  )
   (wire (pts (xy 109.22 114.3) (xy 109.22 115.57))
     (stroke (width 0) (type default) (color 0 0 0 0))
@@
     (stroke (width 0) (type default) (color 0 0 0 0))
   )
-  (wire (pts (xy 50.8 134.62) (xy 53.975 134.62))
-    (stroke (width 0) (type default) (color 0 0 0 0))
-  )
   (wire (pts (xy 22.86 24.13) (xy 25.4 24.13))
     (stroke (width 0) (type default) (color 0 0 0 0))
   )
-  (wire (pts (xy 90.17 24.765) (xy 90.17 28.575))
-    (stroke (width 0) (type default) (color 0 0 0 0))
-  )
   (wire (pts (xy 136.525 22.86) (xy 136.525 29.21))
     (stroke (width 0) (type default) (color 0 0 0 0))
@@
     (stroke (width 0) (type default) (color 0 0 0 0))
   )
-  (wire (pts (xy 107.95 135.89) (xy 111.76 135.89))
-    (stroke (width 0) (type default) (color 0 0 0 0))
-  )
   (wire (pts (xy 78.74 36.195) (xy 78.74 38.735))
     (stroke (width 0) (type default) (color 0 0 0 0))
@@
     (effects (font (size 1.27 1.27)) (justify right bottom))
   )
-  (label "3V3" (at 115.57 69.85 0)
-    (effects (font (size 1.27 1.27)) (justify left bottom))
-  )
-  (label "3V3" (at 53.975 132.08 0)
-    (effects (font (size 1.27 1.27)) (justify left bottom))
-  )
   (label "ESP_RX" (at 120.65 88.9 0)
     (effects (font (size 1.27 1.27)) (justify left bottom))
@@
     (effects (font (size 1.27 1.27)) (justify right bottom))
   )
-  (label "3V3" (at 90.17 24.765 0)
-    (effects (font (size 1.27 1.27)) (justify left bottom))
-  )
   (label "USB_DN" (at 68.58 84.455 0)
     (effects (font (size 1.27 1.27)) (justify left bottom))
@@
     (effects (font (size 1.27 1.27)) (justify left bottom))
   )
-  (label "5V" (at 53.975 129.54 0)
-    (effects (font (size 1.27 1.27)) (justify left bottom))
-  )
   (label "USB_DP" (at 68.58 86.995 0)
-    (effects (font (size 1.27 1.27)) (justify left bottom))
-  )
-  (label "3V3" (at 107.95 135.89 180)
-    (effects (font (size 1.27 1.27)) (justify right bottom))
-  )
-  (label "3V3" (at 140.97 40.64 0)
     (effects (font (size 1.27 1.27)) (justify left bottom))
   )
@@
     (effects (font (size 1.27 1.27)) (justify left))
   )
-  (hierarchical_label "+3V3" (shape passive) (at 111.76 135.89 0)
-    (effects (font (size 1.27 1.27)) (justify left))
-  )
   (hierarchical_label "ESP_RX" (shape output) (at 111.76 147.32 0)
     (effects (font (size 1.27 1.27)) (justify left))
@@
     (pin "1")
     (pin "2")
+  )
+  (symbol (lib_id "power:+3.3V") (at 140.97 40.64 0) (unit 1)
+    (in_bom yes) (on_board yes)
+    (property "Reference" "#PWR0134" (id 0) (at 140.97 44.45 0)
+      (effects (font (size 1.27 1.27)) hide)
+    )
+    (property "Value" "+3.3V" (id 1) (at 142.24 38.1 0)
+      (effects (font (size 1.27 1.27)) (justify left))
+    )
+    (property "Footprint" "" (id 2) (at 140.97 40.64 0)
+      (effects (font (size 1.27 1.27)) hide)
+    )
+    (property "Datasheet" "" (id 3) (at 140.97 40.64 0)
+      (effects (font (size 1.27 1.27)) hide)
+    )
+    (pin "1")
   )
   (symbol (lib_id "Device:LED") (at 125.095 48.26 0) (unit 1)
@@
     (pin "2")
   )
+  (symbol (lib_id "power:+3.3V") (at 90.17 28.575 0) (unit 1)
+    (in_bom yes) (on_board yes)
+    (property "Reference" "#PWR0142" (id 0) (at 90.17 32.385 0)
+      (effects (font (size 1.27 1.27)) hide)
+    )
+    (property "Value" "+3.3V" (id 1) (at 91.44 26.035 0)
+      (effects (font (size 1.27 1.27)) (justify left))
+    )
+    (property "Footprint" "" (id 2) (at 90.17 28.575 0)
+      (effects (font (size 1.27 1.27)) hide)
+    )
+    (property "Datasheet" "" (id 3) (at 90.17 28.575 0)
+      (effects (font (size 1.27 1.27)) hide)
+    )
+    (pin "1")
+  )
   (symbol (lib_id "Device:R") (at 132.715 48.26 270) (unit 1)
     (in_bom yes) (on_board yes)
@@
     (pin "2")
   )
-  (symbol (lib_id "power:GND") (at 53.975 134.62 90) (unit 1)
-    (in_bom yes) (on_board yes)
-    (property "Reference" "#PWR0134" (id 0) (at 60.325 134.62 0)
-      (effects (font (size 1.27 1.27)) hide)
-    )
-    (property "Value" "GND" (id 1) (at 57.785 134.62 90)
-      (effects (font (size 1.27 1.27)) (justify right))
-    )
-    (property "Footprint" "" (id 2) (at 53.975 134.62 0)
-      (effects (font (size 1.27 1.27)) hide)
-    )
-    (property "Datasheet" "" (id 3) (at 53.975 134.62 0)
-      (effects (font (size 1.27 1.27)) hide)
-    )
-    (pin "1")
-  )
   (symbol (lib_id "Device:R") (at 29.21 38.1 90) (unit 1)
     (in_bom yes) (on_board yes)
@@
     )
     (property "Datasheet" "" (id 3) (at 127 82.55 0)
+      (effects (font (size 1.27 1.27)) hide)
+    )
+    (pin "1")
+  )
+  (symbol (lib_id "power:+3.3V") (at 115.57 69.85 0) (unit 1)
+    (in_bom yes) (on_board yes)
+    (property "Reference" "#PWR0115" (id 0) (at 115.57 73.66 0)
+      (effects (font (size 1.27 1.27)) hide)
+    )
+    (property "Value" "+3.3V" (id 1) (at 116.84 67.31 0)
+      (effects (font (size 1.27 1.27)) (justify left))
+    )
+    (property "Footprint" "" (id 2) (at 115.57 69.85 0)
+      (effects (font (size 1.27 1.27)) hide)
+    )
+    (property "Datasheet" "" (id 3) (at 115.57 69.85 0)
       (effects (font (size 1.27 1.27)) hide)
     )
@@
     (pin "2")
   )
-  (sheet (at 38.1 128.27) (size 12.7 7.62) (fields_autoplaced)
-    (stroke (width 0.1524) (type solid) (color 0 0 0 0))
-    (fill (color 0 0 0 0.0000))
-    (property "Sheet name" "AMS1117-5V-3v3" (id 0) (at 38.1 127.5584 0)
-      (effects (font (size 1.27 1.27)) (justify left bottom))
-    )
-    (property "Sheet file" "voltage_regulator.kicad_sch" (id 1) (at 38.1 136.4746 0)
-      (effects (font (size 1.27 1.27)) (justify left top))
-    )
-    (pin "5V" bidirectional (at 50.8 129.54 0)
-      (effects (font (size 1.27 1.27)) (justify right))
-    )
-    (pin "GND" bidirectional (at 50.8 134.62 0)
-      (effects (font (size 1.27 1.27)) (justify right))
-    )
-    (pin "3V3" bidirectional (at 50.8 132.08 0)
-      (effects (font (size 1.27 1.27)) (justify right))
-    )
-  )
 )

Commit message: Updated production files
Parts:
- C3, C5: LCSC (none) -> C1525
- C4: LCSC (none) -> C15849
- C6: LCSC (none) -> C19702
- Q2, Q3: LCSC (none) -> C2150
- USBC1: LCSC (none) -> C136423
Changed lines of the file:
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@@
+      (effects (font (size 1.27 1.27)) hide)
+    )
+    (property "LCSC" "C19702" (id 5) (at 164.465 40.005 0)
       (effects (font (size 1.27 1.27)) hide)
     )
@@
       (effects (font (size 1.27 1.27)) hide)
     )
+    (property "LCSC" "C15849" (id 5) (at 93.98 32.385 0)
+      (effects (font (size 1.27 1.27)) hide)
+    )
     (pin "1")
     (pin "2")
@@
     (property "JLC Part" "Basic Part" (id 6) (at 44.45 38.1 0)
       (effects (font (size 0 0)) hide)
+    )
+    (property "LCSC" "C2150" (id 7) (at 45.72 36.83 0)
+      (effects (font (size 1.27 1.27)) hide)
     )
     (pin "1")
@@
       (effects (font (size 1.27 1.27)) hide)
     )
+    (property "LCSC" "C1525" (id 5) (at 123.19 77.47 0)
+      (effects (font (size 1.27 1.27)) hide)
+    )
     (pin "1")
     (pin "2")
@@
     (property "JLC Part" "Extended Part" (id 6) (at 55.88 80.645 0)
       (effects (font (size 0 0)) hide)
+    )
+    (property "LCSC" "C136423" (id 7) (at 55.88 104.775 0)
+      (effects (font (size 1.27 1.27)) hide)
     )
     (pin "1")
@@
       (effects (font (size 0 0)) hide)
     )
+    (property "LCSC" "C2150" (id 7) (at 45.72 22.86 0)
+      (effects (font (size 1.27 1.27)) hide)
+    )
     (pin "1")
     (pin "2")
@@
       (effects (font (size 1.27 1.27)) hide)
     )
+    (property "LCSC" "C1525" (id 5) (at 82.55 34.925 0)
+      (effects (font (size 1.27 1.27)) hide)
+    )
