File: kicad/obs-studio-controller/voltage_regulator.kicad_sch (KiCad schematic)
At the start: 5 parts

Commit message: Placed parts in pcb layout, nothing moved yet
Parts:
- gave numbers to parts that had none: 5
Changed lines of the file:
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@@
   (symbol (lib_id "Device:C") (at 80.01 35.56 180) (unit 1)
     (in_bom yes) (on_board yes)
-    (property "Reference" "C?" (id 0) (at 76.2 35.56 90))
+    (property "Reference" "C10" (id 0) (at 76.2 35.56 90))
     (property "Value" "100n" (id 1) (at 83.82 35.56 90))
     (property "Footprint" "Capacitor_SMD:C_0402_1005Metric" (id 2) (at 79.0448 31.75 0)
@@
   (symbol (lib_id "power:GND") (at 38.1 39.37 0) (unit 1)
     (in_bom yes) (on_board yes) (fields_autoplaced)
-    (property "Reference" "#PWR?" (id 0) (at 38.1 45.72 0)
+    (property "Reference" "#PWR0136" (id 0) (at 38.1 45.72 0)
       (effects (font (size 1.27 1.27)) hide)
     )
@@
   (symbol (lib_id "power:GND") (at 101.6 44.45 270) (unit 1)
     (in_bom yes) (on_board yes)
-    (property "Reference" "#PWR?" (id 0) (at 95.25 44.45 0)
+    (property "Reference" "#PWR0138" (id 0) (at 95.25 44.45 0)
       (effects (font (size 1.27 1.27)) hide)
     )
@@
   (symbol (lib_id "Regulator_Linear:AMS1117-3.3") (at 53.34 30.48 0) (unit 1)
     (in_bom yes) (on_board yes) (fields_autoplaced)
-    (property "Reference" "U?" (id 0) (at 53.34 22.86 0))
+    (property "Reference" "U5" (id 0) (at 53.34 22.86 0))
     (property "Value" "AMS1117-3.3" (id 1) (at 53.34 25.4 0))
     (property "Footprint" "Package_TO_SOT_SMD:SOT-223-3_TabPin2" (id 2) (at 53.34 25.4 0)
@@
   (symbol (lib_id "Device:C") (at 38.1 35.56 180) (unit 1)
     (in_bom yes) (on_board yes)
-    (property "Reference" "C?" (id 0) (at 31.75 35.56 90))
+    (property "Reference" "C8" (id 0) (at 31.75 35.56 90))
     (property "Value" "10u" (id 1) (at 34.29 35.56 90))
     (property "Footprint" "Capacitor_SMD:C_0603_1608Metric" (id 2) (at 37.1348 31.75 0)
@@
   (symbol (lib_id "Device:C") (at 68.58 35.56 0) (unit 1)
     (in_bom yes) (on_board yes)
-    (property "Reference" "C?" (id 0) (at 74.93 35.56 90))
+    (property "Reference" "C9" (id 0) (at 74.93 35.56 90))
     (property "Value" "10u" (id 1) (at 72.39 35.56 90))
     (property "Footprint" "Capacitor_SMD:C_0603_1608Metric" (id 2) (at 69.5452 39.37 0)
@@
   (symbol (lib_id "power:GND") (at 68.58 39.37 0) (unit 1)
     (in_bom yes) (on_board yes) (fields_autoplaced)
-    (property "Reference" "#PWR?" (id 0) (at 68.58 45.72 0)
+    (property "Reference" "#PWR0135" (id 0) (at 68.58 45.72 0)
       (effects (font (size 1.27 1.27)) hide)
     )
@@
   (symbol (lib_id "power:GND") (at 53.34 39.37 0) (unit 1)
     (in_bom yes) (on_board yes) (fields_autoplaced)
-    (property "Reference" "#PWR?" (id 0) (at 53.34 45.72 0)
+    (property "Reference" "#PWR0137" (id 0) (at 53.34 45.72 0)
       (effects (font (size 1.27 1.27)) hide)
     )
@@
   (symbol (lib_id "Device:C") (at 26.67 35.56 180) (unit 1)
     (in_bom yes) (on_board yes)
-    (property "Reference" "C?" (id 0) (at 22.86 35.56 90))
+    (property "Reference" "C7" (id 0) (at 22.86 35.56 90))
     (property "Value" "100n" (id 1) (at 30.48 35.56 90))
     (property "Footprint" "Capacitor_SMD:C_0402_1005Metric" (id 2) (at 25.7048 31.75 0)

Commit message: Routing complete
Connections:
- net 3V3 renamed +3V3
Changed lines of the file:
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@@
-    (stroke (width 0) (type default) (color 0 0 0 0))
-  )
-  (wire (pts (xy 99.06 41.275) (xy 101.6 41.275))
     (stroke (width 0) (type default) (color 0 0 0 0))
   )
@@
     (effects (font (size 1.27 1.27)) (justify right bottom))
   )
-  (label "3V3" (at 68.58 27.94 0)
-    (effects (font (size 1.27 1.27)) (justify left bottom))
-  )
-  (label "3V3" (at 99.06 41.275 180)
-    (effects (font (size 1.27 1.27)) (justify right bottom))
-  )
   (hierarchical_label "GND" (shape bidirectional) (at 101.6 44.45 0)
     (effects (font (size 1.27 1.27)) (justify left))
   )
   (hierarchical_label "5V" (shape bidirectional) (at 101.6 47.625 0)
-    (effects (font (size 1.27 1.27)) (justify left))
-  )
-  (hierarchical_label "3V3" (shape bidirectional) (at 101.6 41.275 0)
     (effects (font (size 1.27 1.27)) (justify left))
   )
@@
   (symbol (lib_id "power:GND") (at 38.1 39.37 0) (unit 1)
     (in_bom yes) (on_board yes) (fields_autoplaced)
-    (property "Reference" "#PWR0136" (id 0) (at 38.1 45.72 0)
+    (property "Reference" "#PWR0140" (id 0) (at 38.1 45.72 0)
       (effects (font (size 1.27 1.27)) hide)
     )
@@
     (pin "2")
   )
+  (symbol (lib_id "power:+3.3V") (at 68.58 27.94 0) (unit 1)
+    (in_bom yes) (on_board yes)
+    (property "Reference" "#PWR0143" (id 0) (at 68.58 31.75 0)
+      (effects (font (size 1.27 1.27)) hide)
+    )
+    (property "Value" "+3.3V" (id 1) (at 63.5 24.13 0)
+      (effects (font (size 1.27 1.27)) (justify left))
+    )
+    (property "Footprint" "" (id 2) (at 68.58 27.94 0)
+      (effects (font (size 1.27 1.27)) hide)
+    )
+    (property "Datasheet" "" (id 3) (at 68.58 27.94 0)
+      (effects (font (size 1.27 1.27)) hide)
+    )
+    (pin "1")
+  )
   (symbol (lib_id "power:GND") (at 68.58 39.37 0) (unit 1)
     (in_bom yes) (on_board yes) (fields_autoplaced)
-    (property "Reference" "#PWR0135" (id 0) (at 68.58 45.72 0)
+    (property "Reference" "#PWR0141" (id 0) (at 68.58 45.72 0)
       (effects (font (size 1.27 1.27)) hide)
     )

Commit message: Updated production files
Parts:
- C10, C7: LCSC (none) -> C1525
- C8, C9: LCSC (none) -> C19702
Changed lines of the file:
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@@
+      (effects (font (size 1.27 1.27)) hide)
+    )
+    (property "LCSC" "C1525" (id 5) (at 76.2 35.56 0)
       (effects (font (size 1.27 1.27)) hide)
     )
@@
       (effects (font (size 1.27 1.27)) hide)
     )
+    (property "LCSC" "C19702" (id 5) (at 31.75 35.56 0)
+      (effects (font (size 1.27 1.27)) hide)
+    )
     (pin "1")
     (pin "2")
@@
     )
     (property "LCSC Part #" "C19702" (id 4) (at 68.58 35.56 90)
+      (effects (font (size 1.27 1.27)) hide)
+    )
+    (property "LCSC" "C19702" (id 5) (at 74.93 35.56 0)
       (effects (font (size 1.27 1.27)) hide)
     )
@@
       (effects (font (size 1.27 1.27)) hide)
     )
+    (property "LCSC" "C1525" (id 5) (at 22.86 35.56 0)
+      (effects (font (size 1.27 1.27)) hide)
+    )
